File: MPPT.sch (KiCad schematic (older format))
At the start: 0 parts

Commit message: Upd
Parts:
- added C? (x4): CP, symbol CP
- added C? (x2): C, symbol C
- added D? (x2): D_Schottky_Small, symbol D_Schottky_Small
- added L?: INDUCTOR, symbol INDUCTOR
- added P?: PV, symbol CONN_01X02
- added P?: BATT, symbol CONN_01X02
- added Q? (x2): IRFZ44, symbol Q_NMOS_GDS
- added Q? (x2): IRF5305, symbol Q_PMOS_GDS
- added R? (x2): R, symbol R
Connections:
- net labels added: BATT+, BATT-, BOOST_N_GATE, BOOST_P_GATE, BUCK_N_GATE, BUCK_P_Gate, GNDA, Iin+, Iin-, Iout+, Iout-
- wire segments 0 -> 42
